File: POE_tryout.sch (KiCad schematic (older format))
At the start: 0 parts

Commit message: update,
Changed lines of the file:
@@
 $Descr A4 11693 8268
 encoding utf-8
-Sheet 1 2
+Sheet 1 3
 Title ""
 Date ""
@@
 F1 "Si3402.sch" 50
 $EndSheet
+$Sheet
+S 7400 5650 1100 700
+U 5C05912A
+F0 "USB_CH340T" 50
+F1 "USB_CH340T.sch" 50
+$EndSheet
 $EndSCHEMATC
