File: Si3402.sch (KiCad schematic (older format))
At the start: 20 parts, among them U1 Si3402-B-GM

Commit message: update,
Parts:
- C1: footprint (none) -> Capacitor_SMD:C_1206_3216Metric_Pad1.42x1.75mm_HandSolder
Changed lines of the file:
@@
 EESchema Schematic File Version 4
+LIBS:POE_tryout-cache
 EELAYER 26 0
 EELAYER END
@@
 $EndComp
 $Comp
-L taobao-c:C225,1206 C1
-U 1 1 5C006163
-P 2150 1950
-F 0 "C1" H 2250 2000 50  0000 L CNN
-F 1 "C225,1206" H 2250 1950 50  0000 L CNN
-F 2 "" H 2150 1950 50  0001 C CNN
-F 3 "~" H 2150 1950 50  0001 C CNN
-	1    2150 1950
-	1    0    0    -1
-$EndComp
-$Comp
 L taobao-cp:CP1000uf,10V C2
 U 1 1 5C006317
@@
 	9500 1550 9500 1700
 Connection ~ 9500 1700
+$Comp
+L taobao-c:C225,1206 C1
+U 1 1 5C045FF5
+P 2150 1950
+F 0 "C1" H 2250 2000 50  0000 L CNN
+F 1 "C225,1206" H 2250 1950 50  0000 L CNN
+F 2 "Capacitor_SMD:C_1206_3216Metric_Pad1.42x1.75mm_HandSolder" H 2150 1950 50  0001 C CNN
+F 3 "~" H 2150 1950 50  0001 C CNN
+	1    2150 1950
+	1    0    0    -1
+$EndComp
 $EndSCHEMATC

Commit message: update,
Parts:
- removed C5: C226,0805, symbol taobao-c:C226,0805
- added C?: C226,6.3v,0603, Capacitor_SMD:C_0603_1608Metric_Pad1.05x0.95mm_HandSolder, symbol taobao-c:C226,6.3v,0603
Connections:
- net +5VP: now also C?.1
- net at FB1.1, R3.2, R4.2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: now also C?.2
Changed lines of the file:
@@
 $Descr A4 11693 8268
 encoding utf-8
-Sheet 2 2
+Sheet 2 3
 Title ""
 Date ""
@@
 U 1 1 5C005EAF
 P 5350 2750
+AR Path="/5C0031F9/5C005EAF" Ref="U1"  Part="1"
+AR Path="/5C05912A/5C005EAF" Ref="U?"  Part="1"
 F 0 "U1" H 5350 3550 50  0000 C CNN
 F 1 "Si3402-B-GM" H 5350 3450 50  0000 C CNN
@@
 U 1 1 5C006317
 P 3050 1950
+AR Path="/5C0031F9/5C006317" Ref="C2"  Part="1"
+AR Path="/5C05912A/5C006317" Ref="C?"  Part="1"
 F 0 "C2" H 3150 2000 50  0000 L CNN
 F 1 "CP1000uf,10V" H 3150 1950 50  0000 L CNN
@@
 U 1 1 5C006577
 P 2450 2250
+AR Path="/5C0031F9/5C006577" Ref="C4"  Part="1"
+AR Path="/5C05912A/5C006577" Ref="C?"  Part="1"
 F 0 "C4" V 2200 2250 50  0000 C CNN
 F 1 "C104,0603" V 2300 2250 50  0000 C CNN
@@
 U 1 1 5C006717
 P 2450 2550
+AR Path="/5C0031F9/5C006717" Ref="C6"  Part="1"
+AR Path="/5C05912A/5C006717" Ref="C?"  Part="1"
 F 0 "C6" V 2600 2550 50  0000 C CNN
 F 1 "C102,0603" V 2700 2550 50  0000 C CNN
@@
 U 1 1 5C0069E4
 P 3250 2550
+AR Path="/5C0031F9/5C0069E4" Ref="R5"  Part="1"
+AR Path="/5C05912A/5C0069E4" Ref="R?"  Part="1"
 F 0 "R5" V 3000 2550 50  0000 C CNN
 F 1 "R473,0603" V 3100 2550 50  0000 C CNN
@@
 U 1 1 5C007182
 P 3750 3700
+AR Path="/5C0031F9/5C007182" Ref="R7"  Part="1"
+AR Path="/5C05912A/5C007182" Ref="R?"  Part="1"
 F 0 "R7" V 3500 3700 50  0000 C CNN
 F 1 "R49R9,0603" V 3600 3700 50  0000 C CNN
@@
 U 1 1 5C0073B5
 P 2000 4000
+AR Path="/5C0031F9/5C0073B5" Ref="#PWR0101"  Part="1"
+AR Path="/5C05912A/5C0073B5" Ref="#PWR?"  Part="1"
 F 0 "#PWR0101" H 2000 3750 50  0001 C CNN
 F 1 "GND" H 2050 3800 50  0000 C CNN
@@
 U 1 1 5C007A46
 P 2000 2850
+AR Path="/5C0031F9/5C007A46" Ref="C7"  Part="1"
+AR Path="/5C05912A/5C007A46" Ref="C?"  Part="1"
 F 0 "C7" H 1900 2900 50  0000 R CNN
 F 1 "C104,0603" H 1900 2850 50  0000 R CNN
@@
 U 1 1 5C007EE4
 P 9500 1550
+AR Path="/5C0031F9/5C007EE4" Ref="#PWR0102"  Part="1"
+AR Path="/5C05912A/5C007EE4" Ref="#PWR?"  Part="1"
 F 0 "#PWR0102" H 9500 1400 50  0001 C CNN
 F 1 "+5VP" H 9550 1750 50  0000 C CNN
@@
 U 1 1 5C00971B
 P 6650 2050
+AR Path="/5C0031F9/5C00971B" Ref="R1"  Part="1"
+AR Path="/5C05912A/5C00971B" Ref="R?"  Part="1"
 F 0 "R1" H 6750 2100 50  0000 L CNN
 F 1 "25.5k,0603" H 6750 2050 50  0000 L CNN
@@
 $EndComp
 $Comp
-L taobao-c:C226,0805 C5
-U 1 1 5C009D37
-P 9500 2500
-F 0 "C5" H 9600 2550 50  0000 L CNN
-F 1 "C226,0805" H 9600 2500 50  0000 L CNN
-F 2 "" H 9500 2500 50  0001 C CNN
-F 3 "~" H 9500 2500 50  0001 C CNN
-	1    9500 2500
-	1    0    0    -1
-$EndComp
-$Comp
 L taobao-r:R221,1206 R4
 U 1 1 5C00A64A
 P 8950 2500
+AR Path="/5C0031F9/5C00A64A" Ref="R4"  Part="1"
+AR Path="/5C05912A/5C00A64A" Ref="R?"  Part="1"
 F 0 "R4" H 9050 2550 50  0000 L CNN
 F 1 "R221,1206" H 9050 2500 50  0000 L CNN
@@
 U 1 1 5C00A714
 P 8650 2500
+AR Path="/5C0031F9/5C00A714" Ref="R3"  Part="1"
+AR Path="/5C05912A/5C00A714" Ref="R?"  Part="1"
 F 0 "R3" H 8750 2550 50  0000 L CNN
 F 1 "R221,1206" H 8750 2500 50  0000 L CNN
@@
 U 1 1 5C00A8AD
 P 8150 2050
+AR Path="/5C0031F9/5C00A8AD" Ref="R2"  Part="1"
+AR Path="/5C05912A/5C00A8AD" Ref="R?"  Part="1"
 F 0 "R2" H 8250 2100 50  0000 L CNN
 F 1 "R103,0603" H 8250 2050 50  0000 L CNN
@@
 U 1 1 5C00A978
 P 8150 2700
+AR Path="/5C0031F9/5C00A978" Ref="R6"  Part="1"
+AR Path="/5C05912A/5C00A978" Ref="R?"  Part="1"
 F 0 "R6" H 8250 2750 50  0000 L CNN
 F 1 "R303,0603" H 8250 2700 50  0000 L CNN
@@
 U 1 1 5C00FBC6
 P 7750 2950
+AR Path="/5C0031F9/5C00FBC6" Ref="FB1"  Part="1"
+AR Path="/5C05912A/5C00FBC6" Ref="FB?"  Part="1"
 F 0 "FB1" V 7500 2950 50  0000 C CNN
 F 1 "R600, 0805, 2A" V 7600 2950 50  0000 C CNN
@@
 U 1 1 5C00FCFF
 P 7300 2950
+AR Path="/5C0031F9/5C00FCFF" Ref="L1"  Part="1"
+AR Path="/5C05912A/5C00FCFF" Ref="L?"  Part="1"
 F 0 "L1" V 7500 2950 50  0000 C CNN
 F 1 "L_33uH" V 7400 2950 50  0000 C CNN
@@
 U 1 1 5C013D82
 P 7500 2150
+AR Path="/5C0031F9/5C013D82" Ref="C3"  Part="1"
+AR Path="/5C05912A/5C013D82" Ref="C?"  Part="1"
 F 0 "C3" H 7600 2200 50  0000 L CNN
 F 1 "CP_Small" H 7600 2150 50  0000 L CNN
@@
 U 1 1 5C013F1D
 P 6950 2150
+AR Path="/5C0031F9/5C013F1D" Ref="D1"  Part="1"
+AR Path="/5C05912A/5C013F1D" Ref="D?"  Part="1"
 F 0 "D1" V 6900 2250 50  0000 L CNN
 F 1 "D_Zener_Small" V 6950 2250 50  0000 L CNN
@@
 U 1 1 5C01B407
 P 6600 3850
+AR Path="/5C0031F9/5C01B407" Ref="JP1"  Part="1"
+AR Path="/5C05912A/5C01B407" Ref="JP?"  Part="1"
 F 0 "JP1" H 6600 4050 50  0000 C CNN
 F 1 "Jumper_NO_Small" H 6600 3950 50  0000 C CNN
@@
 U 1 1 5C01B481
 P 6600 3950
+AR Path="/5C0031F9/5C01B481" Ref="JP2"  Part="1"
+AR Path="/5C05912A/5C01B481" Ref="JP?"  Part="1"
 F 0 "JP2" H 6600 4150 50  0000 C CNN
 F 1 "Jumper_NO_Small" H 6600 4050 50  0000 C CNN
@@
 U 1 1 5C045FF5
 P 2150 1950
+AR Path="/5C0031F9/5C045FF5" Ref="C1"  Part="1"
+AR Path="/5C05912A/5C045FF5" Ref="C?"  Part="1"
 F 0 "C1" H 2250 2000 50  0000 L CNN
 F 1 "C225,1206" H 2250 1950 50  0000 L CNN
@@
 	1    0    0    -1
 $EndComp
+$Comp
+L taobao-c:C226,6.3v,0603 C?
+U 1 1 5C05AC53
+P 9500 2500
+F 0 "C?" H 9600 2550 50  0000 L CNN
+F 1 "C226,6.3v,0603" H 9600 2500 50  0000 L CNN
+F 2 "Capacitor_SMD:C_0603_1608Metric_Pad1.05x0.95mm_HandSolder" H 9500 2500 50  0001 C CNN
+F 3 "~" H 9500 2500 50  0001 C CNN
+	1    9500 2500
+	1    0    0    -1
+$EndComp
